Commit message: urdf work

File: src/startbot/description/robdesc.urdf.xacro (robot description, xacro)
@@ -9,4 +9,7 @@
 <material name="blue">
     <color rgba="0 0 1 1"/>
+</material>
+<material name="black">
+    <color rgba="0 0 0 1"/>
 </material>
 <link name="base_link">
@@ -56,3 +59,29 @@
 </visual>
 </link>
+<joint name="fcaster_joint" type="fixed">
+<parent link="chassis_link"/>
+<child link="front_caster"/>
+<origin xyz="0.175 0 0"/>
+</joint>
+<link name="front_caster">
+<visual>
+<geometry>
+<sphere radius="0.05"/>
+</geometry>
+<material name="black"/>
+</visual>
+</link>
+<joint name="bcaster_joint" type="fixed">
+<parent link="chassis_link"/>
+<child link="rear_caster"/>
+<origin xyz="-0.175 0 0"/>
+</joint>
+<link name="rear_caster">
+<visual>
+<geometry>
+<sphere radius="0.05"/>
+</geometry>
+<material name="black"/>
+</visual>
+</link>
 </robot>

Commit message: collisions

File: src/startbot/description/robdesc.urdf.xacro (robot description, xacro)
@@ -1,4 +1,31 @@
 <?xml version="1.0"?>
 <robot xmlns:xacro="http://www.ros.org/wiki/xacro" name="startbot">
+<xacro:macro name="inertial_sphere" params="mass radius *origin">
+        <inertial>
+            <xacro:insert_block name="origin"/>
+            <mass value="${mass}" />
+            <inertia ixx="${(2/5) * mass * (radius*radius)}" ixy="0.0" ixz="0.0"
+                    iyy="${(2/5) * mass * (radius*radius)}" iyz="0.0"
+                     izz="${(2/5) * mass * (radius*radius)}" />
+        </inertial>
+    </xacro:macro>
+    <xacro:macro name="inertial_box" params="mass x y z *origin">
+        <inertial>
+            <xacro:insert_block name="origin"/>
+            <mass value="${mass}" />
+            <inertia ixx="${(1/12) * mass * (y*y+z*z)}" ixy="0.0" ixz="0.0"
+                    iyy="${(1/12) * mass * (x*x+z*z)}" iyz="0.0"
+                    izz="${(1/12) * mass * (x*x+y*y)}" />
+        </inertial>
+    </xacro:macro>
+    <xacro:macro name="inertial_cylinder" params="mass length radius *origin">
+        <inertial>
+            <xacro:insert_block name="origin"/>
+            <mass value="${mass}" />
+            <inertia ixx="${(1/12) * mass * (3*radius*radius + length*length)}" ixy="0.0" ixz="0.0"
+                    iyy="${(1/12) * mass * (3*radius*radius + length*length)}" iyz="0.0"
+                    izz="${(1/2) * mass * (radius*radius)}" />
+        </inertial>
+    </xacro:macro>
 <material name="white">
     <color rgba="1 1 1 1"/>
@@ -28,4 +55,10 @@
     <material name="white"/>
 </visual>
+<collision>
+        <origin xyz="0 0 0.075" rpy="0 0 0"/>
+        <geometry>
+        <box size="0.45 0.35 0.15"/>
+        </geometry>
+    </collision>
 </link>
 <!--left wheel-->
@@ -41,4 +74,9 @@
 <cylinder length="0.06" radius="0.05"/>
 </geometry>
+<collision>
+<geometry>
+<cylinder length="0.06" radius="0.05"/>
+</geometry>
+</collision>
 <material name="blue"/>
 </visual>
@@ -58,4 +96,9 @@
 <material name="blue"/>
 </visual>
+<collision>
+<geometry>
+<cylinder length="0.06" radius="0.05"/>
+</geometry>
+</collision>
 </link>
 <joint name="fcaster_joint" type="fixed">
@@ -71,4 +114,9 @@
 <material name="black"/>
 </visual>
+<collision>
+<geometry>
+<sphere radius="0.05"/>
+</geometry>
+</collision>
 </link>
 <joint name="bcaster_joint" type="fixed">
@@ -84,4 +132,9 @@
 <material name="black"/>
 </visual>
+<collision>
+<geometry>
+<sphere radius="0.05"/>
+</geometry>
+</collision>
 </link>
 </robot>

Commit message: inertials

File: src/startbot/description/robdesc.urdf.xacro (robot description, xacro)
@@ -61,4 +61,7 @@
         </geometry>
     </collision>
+    <xacro:inertial_box mass="0.5" x="0.45" y="0.35" z="0.15">
+        <origin xyz="0 0 0.075" rpy="0 0 0"/>
+    </xacro:inertial_box>
 </link>
 <!--left wheel-->
@@ -74,4 +77,6 @@
 <cylinder length="0.06" radius="0.05"/>
 </geometry>
+<material name="blue"/>
+</visual>
 <collision>
 <geometry>
@@ -79,6 +84,7 @@
 </geometry>
 </collision>
-<material name="blue"/>
-</visual>
+    <xacro:inertial_cylinder mass="0.1" length="0.06" radius="0.05">
+        <origin xyz="0 0 0" rpy="0 0 0"/>
+    </xacro:inertial_cylinder>
 </link>
 <!--right wheel-->
@@ -101,4 +107,7 @@
 </geometry>
 </collision>
+    <xacro:inertial_cylinder mass="0.1" length="0.06" radius="0.05">
+        <origin xyz="0 0 0" rpy="0 0 0"/>
+    </xacro:inertial_cylinder>
 </link>
 <joint name="fcaster_joint" type="fixed">
@@ -119,4 +128,7 @@
 </geometry>
 </collision>
+    <xacro:inertial_sphere mass="0.1" radius="0.05">
+        <origin xyz="0 0 0" rpy="0 0 0"/>
+    </xacro:inertial_sphere>
 </link>
 <joint name="bcaster_joint" type="fixed">
@@ -137,4 +149,7 @@
 </geometry>
 </collision>
+    <xacro:inertial_sphere mass="0.1" radius="0.05">
+        <origin xyz="0 0 0" rpy="0 0 0"/>
+    </xacro:inertial_sphere>
 </link>
 </robot>

Commit message: gazebo integration

File: src/startbot/description/robdesc.urdf.xacro (robot description, xacro)
@@ -65,4 +65,7 @@
     </xacro:inertial_box>
 </link>
+<gazebo reference="chassis_link">
+<material>Gazebo/White</material>
+</gazebo>
 <!--left wheel-->
 <joint name="left_joint" type="continuous">
@@ -88,4 +91,7 @@
     </xacro:inertial_cylinder>
 </link>
+<gazebo reference="left_wheel">
+<material>Gazebo/Blue</material>
+</gazebo>
 <!--right wheel-->
 <joint name="right_joint" type="continuous">
@@ -111,4 +117,8 @@
     </xacro:inertial_cylinder>
 </link>
+<gazebo reference="right_wheel">
+<material>Gazebo/Blue</material>
+</gazebo>
+<!-- caster wheels-->
 <joint name="fcaster_joint" type="fixed">
 <parent link="chassis_link"/>
@@ -132,4 +142,9 @@
     </xacro:inertial_sphere>
 </link>
+<gazebo reference="front_caster">
+<material>Gazebo/Black</material>
+<mu1 value="0.0001"/>
+<mu2 value="0.0001"/>
+</gazebo>
 <joint name="bcaster_joint" type="fixed">
 <parent link="chassis_link"/>
@@ -153,3 +168,8 @@
     </xacro:inertial_sphere>
 </link>
+<gazebo reference="rear_caster">
+<material>Gazebo/Black</material>
+<mu1 value="0.0001"/>
+<mu2 value="0.0001"/>
+</gazebo>
 </robot>
